File: PowerLossHeatCreepArrester_v1.0/PowerLossHeatCreepArrester_v1.0.kicad_pcb (KiCad board)
At the start: 2 copper layers, 62 x 41 mm, 57 parts, among them J1 Conn_01x04_Socket, J2 BC3550Y0302A, J3 Conn_01x04_Pin, Q1 BSS138, Q2 BSS138, U1 LM393, U2 MT3608, U3 TP4056-42-ESOP8, U5 MP1584EN

Commit message: rev_1.0: independent temperature sensing, comparator divider redesign
Hardware changes:
- Add U4: independent temperature monitoring IC with dedicated thermistor.
  Sharing the printer's NTC directly with this board is not feasible without
  a 3.3 V interface solution; U4 provides an isolated temperature signal to
  LM393 comparator 2 for the > 50 °C fan activation threshold.

Schematic (kicad_sch):
- Recalculate comparator 1 (power-loss) voltage divider:
    R15: 210k → 52.3k
    R16: 40.2k → 10k
- Update hysteresis / reference network:
    R21: 200k → 100k
    Comparator reference resistors: 10k → 47k and 10k → 910k
- Reroute GND symbol and reposition thermistor net label for clarity
- Add schematic note documenting the thermistor isolation decision
- Fix net label typo: 'indipendent' → 'independent'
- Minor wording update in annotation text (package → chip)

PCB layout (kicad_pcb):
- Place U4 footprint at (138.51, 88.06, 90°) on F.Cu
- Update net assignments on affected pads to match schematic
- Set solder_mask_to_copper_clearance: 0.0 → 0.005 mm
- Add back-silkscreen label and minor component placement adjustments

Project file (kicad_pro):
- Record U4 in used_designators
- Persist updated DRC constraint (solder mask clearance 0.005 mm)

Documentation (README.md):
- Add Independent temperature monitoring row to Design Notes table
- Add Revision History section summarising rev_1.0 changes

Co-authored-by: Copilot <223556219+Copilot@users.noreply.github.com>
Parts:
- added REF**: R_Axial_DIN0204_L3.6mm_D1.6mm_P7.62mm_Horizontal, Resistor_THT:R_Axial_DIN0204_L3.6mm_D1.6mm_P7.62mm_Horizontal, F.Cu at (138.5, 88.1)

Commit message: rev_1.0: add Q3 reverse protection on fan control input
- Q3 (ZXMP6A13FTA, SOT-23, P-ch): placed on 'independent_3d printer
  fan control input' net at (22.86, 88.9)
  Source = fan control rail, Drain = protected node, Gate = GND via R23
- R23 (10k, 0603): gate pull-down resistor for Q3
  Vgs = -(rail voltage) when correct polarity -> MOSFET fully on
  Reversed polarity -> Vgs = 0 -> MOSFET off, circuit protected
  ZXMP6A13FTA suitable here: signal/control line, negligible current
- Schematic note retained: 24V input and battery side protection
  still to be implemented (ZXMP6A13FTA for 24V, AO3401A for battery)
- PCB layout and project file updated to match

Co-authored-by: Copilot <223556219+Copilot@users.noreply.github.com>
Parts:
- removed REF**: R_Axial_DIN0204_L3.6mm_D1.6mm_P7.62mm_Horizontal, Resistor_THT:R_Axial_DIN0204_L3.6mm_D1.6mm_P7.62mm_Horizontal
- added 5V1: TestPoint_Alt, TestPoint:TestPoint_Pad_D1.5mm, F.Cu at (129.0, 85.3)
- added GND1: TestPoint_Alt, TestPoint:TestPoint_Pad_D1.5mm, F.Cu at (164.8, 105.2)
- added R22: 100k, Resistor_SMD:R_0603_1608Metric, F.Cu at (133.2, 86.2)
- R10: value 10k -> 910K
- R11: value 10k -> 47k
- R15: value 210k -> 52.3k
- R16: value 40.2k -> 10k
- R21: value 200k -> 100k
Connections:
- D6 pad 2: /24V_from printer power supply -> /indipendent_3d printer fan control input
- J1 pad 1: GND -> /12V_Boosted
Routing:
- net /12V_Boosted: track 85.8 -> 93.6 mm
- net /thermistor input: track 70.4 -> 76.1 mm
- net GND: track 24.6 -> 20.3 mm, vias 63 -> 64
Other:
- board text added: "12V_BOOSTED"
- board text added: "XundaTech Heat Creep Arrester V1.0"
- board text removed: "GND"
- board text removed: "XundaTech Heat Creeep Arrester V1.0"
